Commit message: Changes on URDF for compatibility

File: src/dimitri_description/urdf/dimitri.urdf (robot description, URDF)
Before this commit: robot dimitri, 23 links, 22 joints
Links:
- link root: mass 0.001 -> None
Joints:
- removed joint abdomen_link
- removed joint abdomen_upper_link
- removed joint base_link
- removed joint camera_link
- removed joint head_link
- removed joint left_back_gripper_link
- removed joint left_front_gripper
- removed joint left_hand_link
- removed joint left_shoulder_link
- removed joint left_under_arm_link
- removed joint left_upper_arm_link
- removed joint left_wrist_link
- removed joint neck_link
- removed joint right_back_gripper_link
- removed joint right_front_gripper_link
- removed joint right_hand_link
- removed joint right_shoulder_link
- removed joint right_under_arm_link
- removed joint right_upper_arm_link
- removed joint right_wrist_link
- removed joint torso_link
- removed joint torso_under_link
- added joint abdomen_joint: type revolute, parent base_link, child abdomen_link, origin xyz=-0.01876 0.02798 0.43095 rpy=-1.5708 0 0, axis 0 0 1.0, limit lower=-0.45379 upper=0.45379 effort=10.0 velocity=0.03491
- added joint abdomen_upper_joint: type revolute, parent abdomen_link, child abdomen_upper_link, origin xyz=0.01917 0.00123 -0.02722 rpy=1.5708 0 1.5708, axis 0 0 1.0, limit lower=-0.45379 upper=0.45379 effort=10.0 velocity=0.03491
- added joint base_joint: type fixed, parent root, child base_link, origin xyz=0 0 0.12353 rpy=0 0 0
- added joint camera_joint: type fixed, parent head_link, child camera_link, origin xyz=-0.0085 -0.11925 0.00567 rpy=1.5708 0 0.68865
- added joint head_joint: type revolute, parent neck_link, child head_link, origin xyz=0.00084 -0.0004 0.07009 rpy=0 1.5708 0, axis 0 0 1.0, limit lower=-0.34907 upper=0.2618 effort=10.0 velocity=0.03491
- added joint left_back_gripper_joint: type revolute, parent left_hand_link, child left_back_gripper_link, origin xyz=0.01536 0.09638 -0.00157 rpy=0 0 -1.5708, axis 0 0 1.0, limit lower=0 upper=1.309 effort=10.0 velocity=0.03491
- added joint left_front_gripper_joint: type revolute, parent left_hand_link, child left_front_gripper, origin xyz=-0.01893 0.09638 0.00011 rpy=3.14159 0 -1.5708, axis 0 0 1.0, limit lower=0 upper=1.309 effort=10.0 velocity=0.03491
- added joint left_hand_joint: type revolute, parent left_wrist_link, child left_hand_link, origin xyz=-0.00012 0.001 -0.02198 rpy=-1.5708 0 0, axis 0 0 1.0, limit lower=0 upper=1.5708 effort=10.0 velocity=0.03491
- added joint left_shoulder_joint: type revolute, parent torso_link, child left_shoulder_link, origin xyz=0.01176 0.11735 0.01717 rpy=1.5708 -1.5708 0, axis 0 0 1.0, limit lower=-0.5236 upper=2.61799 effort=10.0 velocity=0.03491
- added joint left_under_arm_joint: type revolute, parent left_upper_arm_link, child left_under_arm_link, origin xyz=0.01456 0.11997 -0.0184 rpy=1.5708 0 1.5708, axis 0 0 1.0, limit lower=0 upper=1.5708 effort=10.0 velocity=0.03491
- added joint left_upper_arm_joint: type revolute, parent left_shoulder_link, child left_upper_arm_link, origin xyz=0.00078 -0.01161 -0.02742 rpy=1.5708 -1.5708 0, axis 0 0 1.0, limit lower=0 upper=2.26893 effort=10.0 velocity=0.03491
- added joint left_wrist_joint: type revolute, parent left_under_arm_link, child left_wrist_link, origin xyz=0.12993 0.00068 -0.00159 rpy=1.5708 0 -1.5708, axis 0 0 1.0, limit lower=0 upper=4.71239 effort=10.0 velocity=0.03491
- added joint neck_joint: type revolute, parent torso_link, child neck_link, origin xyz=-0.00148 0.0012 0.06885 rpy=0 0 1.5708, axis 0 0 1.0, limit lower=-1.0472 upper=1.0472 effort=10.0 velocity=0.03491
- added joint right_back_gripper_joint: type revolute, parent right_hand_link, child right_back_gripper_link, origin xyz=-0.01669 -0.09929 0.00166 rpy=0 0 -1.5708, axis 0 0 1.0, limit lower=0 upper=1.309 effort=10.0 velocity=0.03491
- added joint right_front_gripper_joint: type revolute, parent right_hand_link, child right_front_gripper_link, origin xyz=0.0191 -0.09917 0.00014 rpy=-3.14159 0 -1.5708, axis 0 0 1.0, limit lower=0 upper=1.309 effort=10.0 velocity=0.03491
- added joint right_hand_joint: type revolute, parent right_wrist_link, child right_hand_link, origin xyz=0.00012 0.00225 0.02795 rpy=-1.5708 0 0, axis 0 0 1.0, limit lower=0 upper=1.5708 effort=10.0 velocity=0.03491
- added joint right_shoulder_joint: type revolute, parent torso_link, child right_shoulder_link, origin xyz=0.01176 -0.12018 0.01717 rpy=1.5708 1.5708 0, axis 0 0 1.0, limit lower=-0.5236 upper=2.61799 effort=10.0 velocity=0.03491
- added joint right_under_arm_joint: type revolute, parent right_upper_arm_link, child right_under_arm_link, origin xyz=-0.00738 -0.11596 -5e-05 rpy=0 1.5708 0, axis 0 0 1.0, limit lower=0 upper=1.5708 effort=10.0 velocity=0.03491
- added joint right_upper_arm_joint: type revolute, parent right_shoulder_link, child right_upper_arm_link, origin xyz=0.0001 -0.00679 0.02608 rpy=1.5708 -1.5708 0, axis 0 0 1.0, limit lower=0 upper=2.61799 effort=10.0 velocity=0.03491
- added joint right_wrist_joint: type revolute, parent right_under_arm_link, child right_wrist_link, origin xyz=0.00063 -0.12268 -0.00602 rpy=1.5708 0 0, axis 0 0 1.0, limit lower=0 upper=4.71239 effort=10.0 velocity=0.03491
- added joint torso_joint: type fixed, parent torso_under_link, child torso_link, origin xyz=0.00836 -0.00182 0.08279 rpy=0 0 0
- added joint torso_under_joint: type fixed, parent abdomen_upper_link, child torso_under_link, origin xyz=-0.0901 0.0006 -0.04379 rpy=0 -1.5708 0

Commit message: Added end-factor.

File: src/dimitri_description/urdf/dimitri.urdf (robot description, URDF)
Before this commit: robot dimitri, 23 links, 22 joints
Links:
- added link left_end_factor, mass 0.001
- added link right_end_factor, mass 0.001
Joints:
- added joint left_end_factor_joint: type fixed, parent left_hand_link, child left_end_factor, origin xyz=-0.00288 0.17394 0.00113 rpy=0 -3.14159 0
- added joint right_end_factor_joint: type fixed, parent right_hand_link, child right_end_factor, origin xyz=0.0026 -0.17836 0.00053 rpy=0 0 0

Commit message: textures?

File: src/dimitri_description/urdf/dimitri.urdf (robot description, URDF)
Before this commit: robot dimitri, 25 links, 24 joints
Joints:
- removed joint camera_joint
- added joint camera_link: type fixed, parent head_link, child camera_link, origin xyz=-0.01667 -0.11925 0.00567 rpy=1.5708 0 0.09495
